Commit message: add left ee operator

File: resources/robots/h1_2_arm/h1_2_7dof.urdf (robot description, URDF)
Before this commit: robot h1_5, 56 links, 55 joints
Links:
- removed link L_hand_base_link
- removed link L_index_intermediate
- removed link L_index_proximal
- removed link L_middle_intermediate
- removed link L_middle_proximal
- removed link L_pinky_intermediate
- removed link L_pinky_proximal
- removed link L_ring_intermediate
- removed link L_ring_proximal
- removed link L_thumb_distal
- removed link L_thumb_intermediate
- removed link L_thumb_proximal
- removed link L_thumb_proximal_base
- added link ee_op, mass 0.001; collision sphere radius=0.01
Joints:
- removed joint L_base_link_joint
- removed joint L_index_intermediate_joint
- removed joint L_index_proximal_joint
- removed joint L_middle_intermediate_joint
- removed joint L_middle_proximal_joint
- removed joint L_pinky_intermediate_joint
- removed joint L_pinky_proximal_joint
- removed joint L_ring_intermediate_joint
- removed joint L_ring_proximal_joint
- removed joint L_thumb_distal_joint
- removed joint L_thumb_intermediate_joint
- removed joint L_thumb_proximal_pitch_joint
- removed joint L_thumb_proximal_yaw_joint
- added joint left_wrist_to_ee_op: type fixed, parent left_wrist_yaw_link, child ee_op, origin xyz=0.05 0 0 rpy=0 0 0

Commit message: initialize the contact manipulation RL code

File: resources/robots/h1_2_arm/h1_2_7dof.urdf (robot description, URDF)
Before this commit: robot h1_5, 44 links, 43 joints
Links:
- removed link ee_op
- added link left_ee_op, mass 0.001; collision sphere radius=0.01
Joints:
- joint left_wrist_to_ee_op: child ee_op -> left_ee_op

Commit message: 20251110

File: resources/robots/h1_2_arm/h1_2_7dof.urdf (robot description, URDF)
Before this commit: robot h1_5, 44 links, 43 joints
Joints:
- joint left_elbow_pitch_joint: type revolute -> fixed
- joint left_elbow_roll_joint: type revolute -> fixed
- joint left_shoulder_pitch_joint: type revolute -> fixed
- joint left_shoulder_roll_joint: type revolute -> fixed
- joint left_shoulder_yaw_joint: type revolute -> fixed
- joint left_wrist_pitch_joint: type revolute -> fixed
- joint left_wrist_yaw_joint: type revolute -> fixed

Commit message: 20251111

File: resources/robots/h1_2_arm/h1_2_7dof.urdf (robot description, URDF)
Before this commit: robot h1_5, 44 links, 43 joints
Joints:
- joint left_elbow_pitch_joint: type fixed -> revolute
- joint left_elbow_roll_joint: type fixed -> revolute
- joint left_shoulder_pitch_joint: type fixed -> revolute
- joint left_shoulder_roll_joint: type fixed -> revolute
- joint left_shoulder_yaw_joint: type fixed -> revolute
- joint left_wrist_pitch_joint: type fixed -> revolute
- joint left_wrist_yaw_joint: type fixed -> revolute
- joint right_elbow_pitch_joint: type revolute -> fixed
- joint right_elbow_roll_joint: type revolute -> fixed
- joint right_shoulder_pitch_joint: type revolute -> fixed
- joint right_shoulder_roll_joint: type revolute -> fixed
- joint right_shoulder_yaw_joint: type revolute -> fixed
- joint right_wrist_pitch_joint: type revolute -> fixed
- joint right_wrist_yaw_joint: type revolute -> fixed

Commit message: fix base link

File: resources/robots/h1_2_arm/h1_2_7dof.urdf (robot description, URDF)
Before this commit: robot h1_5, 44 links, 43 joints
Links:
- added link world
Joints:
- added joint fixed_base: type fixed, parent world, child pelvis, origin xyz=0 0 0 rpy=0 0 0

Commit message: remove other parts in urdf, recover end effector model

File: resources/robots/h1_2_arm/h1_2_7dof.urdf (robot description, URDF)
Before this commit: robot h1_5, 45 links, 44 joints
Links:
- removed link R_hand_base_link
- removed link R_index_intermediate
- removed link R_index_proximal
- removed link R_middle_intermediate
- removed link R_middle_proximal
- removed link R_pinky_intermediate
- removed link R_pinky_proximal
- removed link R_ring_intermediate
- removed link R_ring_proximal
- removed link R_thumb_distal
- removed link R_thumb_intermediate
- removed link R_thumb_proximal
- removed link R_thumb_proximal_base
- removed link imu_link
- removed link left_ankle_pitch_link
- removed link left_ankle_roll_link
- removed link left_ee_op
- removed link left_hip_pitch_link
- removed link left_hip_roll_link
- removed link left_hip_yaw_link
- removed link left_knee_link
- removed link logo_link
- removed link pelvis
- removed link right_ankle_pitch_link
- removed link right_ankle_roll_link
- removed link right_elbow_pitch_link
- removed link right_elbow_roll_link
- removed link right_hip_pitch_link
- removed link right_hip_roll_link
- removed link right_hip_yaw_link
- removed link right_knee_link
- removed link right_shoulder_pitch_link
- removed link right_shoulder_roll_link
- removed link right_shoulder_yaw_link
- removed link right_wrist_pitch_link
- removed link right_wrist_yaw_link
- added link L_hand_base_link, mass 0.14143; visual mesh filename=meshes/L_hand_base_link.STL
- added link L_index_intermediate, mass 0.0045682; visual mesh filename=meshes/link16_L.STL
- added link L_index_proximal, mass 0.0042405; visual mesh filename=meshes/link15_L.STL
- added link L_middle_intermediate, mass 0.0050397; visual mesh filename=meshes/link18_L.STL
- added link L_middle_proximal, mass 0.0042405; visual mesh filename=meshes/link17_L.STL
- added link L_pinky_intermediate, mass 0.0036036; visual mesh filename=meshes/link22_L.STL
- added link L_pinky_proximal, mass 0.0042405; visual mesh filename=meshes/link21_L.STL
- added link L_ring_intermediate, mass 0.0045682; visual mesh filename=meshes/link20_L.STL
- added link L_ring_proximal, mass 0.0042405; visual mesh filename=meshes/link19_L.STL
- added link L_thumb_distal, mass 0.003344; visual mesh filename=meshes/link14_L.STL
- added link L_thumb_intermediate, mass 0.0037844; visual mesh filename=meshes/link13_L.STL
- added link L_thumb_proximal, mass 0.0066101; visual mesh filename=meshes/link12_L.STL
- added link L_thumb_proximal_base, mass 0.0018869; visual mesh filename=meshes/link11_L.STL
Joints:
- removed joint R_base_link_joint
- removed joint R_index_intermediate_joint
- removed joint R_index_proximal_joint
- removed joint R_middle_intermediate_joint
- removed joint R_middle_proximal_joint
- removed joint R_pinky_intermediate_joint
- removed joint R_pinky_proximal_joint
- removed joint R_ring_intermediate_joint
- removed joint R_ring_proximal_joint
- removed joint R_thumb_distal_joint
- removed joint R_thumb_intermediate_joint
- removed joint R_thumb_proximal_pitch_joint
- removed joint R_thumb_proximal_yaw_joint
- removed joint imu_joint
- removed joint left_ankle_pitch_joint
- removed joint left_ankle_roll_joint
- removed joint left_hip_pitch_joint
- removed joint left_hip_roll_joint
- removed joint left_hip_yaw_joint
- removed joint left_knee_joint
- removed joint left_wrist_to_ee_op
- removed joint logo_joint
- removed joint right_ankle_pitch_joint
- removed joint right_ankle_roll_joint
- removed joint right_elbow_pitch_joint
- removed joint right_elbow_roll_joint
- removed joint right_hip_pitch_joint
- removed joint right_hip_roll_joint
- removed joint right_hip_yaw_joint
- removed joint right_knee_joint
- removed joint right_shoulder_pitch_joint
- removed joint right_shoulder_roll_joint
- removed joint right_shoulder_yaw_joint
- removed joint right_wrist_pitch_joint
- removed joint right_wrist_yaw_joint
- removed joint torso_joint
- added joint L_base_link_joint: type fixed, parent left_wrist_yaw_link, child L_hand_base_link, origin xyz=0.054 0 0 rpy=0 0 1.5707963267948966192313216916398
- added joint L_index_intermediate_joint: type fixed, parent L_index_proximal, child L_index_intermediate, origin xyz=-0.0024229 -0.032041 -0.001 rpy=0 0 0, axis 0 0 -1, limit lower=0 upper=1.7 effort=1 velocity=0.5, mimic joint=L_index_proximal_joint multiplier=1 offset=0
- added joint L_index_proximal_joint: type fixed, parent L_hand_base_link, child L_index_proximal, origin xyz=0.00028533 -0.13653 0.032268 rpy=-0.034907 0 0, axis 0 0 -1, limit lower=0 upper=1.7 effort=1 velocity=0.5
- added joint L_middle_intermediate_joint: type fixed, parent L_middle_proximal, child L_middle_intermediate, origin xyz=-0.0024229 -0.032041 -0.001 rpy=0 0 0, axis 0 0 -1, limit lower=0 upper=1.7 effort=1 velocity=0.5, mimic joint=L_middle_proximal_joint multiplier=1 offset=0
- added joint L_middle_proximal_joint: type fixed, parent L_hand_base_link, child L_middle_proximal, origin xyz=0.00028533 -0.1371 0.01295 rpy=0 0 0, axis 0 0 -1, limit lower=0 upper=1.7 effort=1 velocity=0.5
- added joint L_pinky_intermediate_joint: type fixed, parent L_pinky_proximal, child L_pinky_intermediate, origin xyz=-0.0024229 -0.032041 -0.001 rpy=0 0 0, axis 0 0 -1, limit lower=0 upper=1.7 effort=1 velocity=0.5, mimic joint=L_pinky_proximal_joint multiplier=1 offset=0
- added joint L_pinky_proximal_joint: type fixed, parent L_hand_base_link, child L_pinky_proximal, origin xyz=0.00028533 -0.13571 -0.025488 rpy=0.10472 0 0, axis 0 0 -1, limit lower=0 upper=1.7 effort=1 velocity=0.5
- added joint L_ring_intermediate_joint: type fixed, parent L_ring_proximal, child L_ring_intermediate, origin xyz=-0.0024229 -0.032041 -0.001 rpy=0 0 0, axis 0 0 -1, limit lower=0 upper=1.7 effort=1 velocity=0.5, mimic joint=L_ring_proximal_joint multiplier=1 offset=0
- added joint L_ring_proximal_joint: type fixed, parent L_hand_base_link, child L_ring_proximal, origin xyz=0.00028533 -0.13691 -0.0062872 rpy=0.05236 0 0, axis 0 0 -1, limit lower=0 upper=1.7 effort=1 velocity=0.5
- added joint L_thumb_distal_joint: type fixed, parent L_thumb_intermediate, child L_thumb_distal, origin xyz=0.020248 -0.010156 -0.0012 rpy=0 0 0, axis 0 0 -1, limit lower=0 upper=1.2 effort=1 velocity=0.5, mimic joint=L_thumb_proximal_pitch_joint multiplier=2.4 offset=0
- added joint L_thumb_intermediate_joint: type fixed, parent L_thumb_proximal, child L_thumb_intermediate, origin xyz=0.04407 -0.034553 -0.0008 rpy=0 0 0, axis 0 0 -1, limit lower=0 upper=0.8 effort=1 velocity=0.5, mimic joint=L_thumb_proximal_pitch_joint multiplier=1.6 offset=0
- added joint L_thumb_proximal_pitch_joint: type fixed, parent L_thumb_proximal_base, child L_thumb_proximal, origin xyz=0.0099867 0.0098242 -0.0089 rpy=-1.5708 0 0.16939, axis 0 0 -1, limit lower=-0.1 upper=0.6 effort=1 velocity=0.5
- added joint L_thumb_proximal_yaw_joint: type fixed, parent L_hand_base_link, child L_thumb_proximal_base, origin xyz=-0.01696 -0.0691 0.02045 rpy=1.5708 -1.5708 0, axis 0 0 1, limit lower=-0.1 upper=1.3 effort=1 velocity=0.5
- joint fixed_base: child pelvis -> torso_link
